File: CAD/Picturestack/uPLC-Panel.kicad_pcb (KiCad board)
At the start: 4 copper layers, 70 x 31.4 mm, 186 parts, among them J1.0 Conn_01x06_Pin, J1.1 Conn_01x06_Pin, J1.2 Conn_01x06_Pin, J2.0 SM12B-GHS-TB(LF)(SN), J2.1 SM12B-GHS-TB(LF)(SN), J2.2 SM12B-GHS-TB(LF)(SN), K1.2 G6K-2F-Y, K2.2 G6K-2F-Y, U1.0 AP63201WU, U1.1 AP63201WU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

Commit message: Feat: Prodrun
Parts:
- C19.0, C20.0: value 1uF -> 0.1uF
- L1.0, L1.1, L1.2: value 6.8uH -> 4.7uH
